Commit message: pcd woes

File: src/hand_e/RobotiqHandeROS2Driver/robotiq_hande_description/urdf/robotiq_hande_gripper.ros2_control.xacro (robot description, xacro)
@@ -5,5 +5,5 @@
       <hardware>
         <xacro:if value="${use_fake_hardware}">
-          <plugin>mock_components/GenericSystem</plugin>
+          <plugin>gz_ros2_control/GazeboSimSystem</plugin>
         </xacro:if>
         <xacro:unless value="${use_fake_hardware}">
@@ -32,11 +32,4 @@
         </state_interface>
       </joint>
-      <joint name="${prefix}robotiq_hande_right_finger_joint">
-        <param name="mimic">robotiq_hande_left_finger_joint</param>
-        <param name="multiplier">1</param>
-        <command_interface name="position" />
-        <state_interface name="position"/>
-        <state_interface name="velocity"/>
-      </joint>
     </ros2_control>
   </xacro:macro>

File: src/hand_e/RobotiqHandeROS2Driver/robotiq_hande_description/urdf/robotiq_hande_gripper.xacro (robot description, xacro)
@@ -6,5 +6,22 @@
   <xacro:include filename="$(find robotiq_hande_description)/urdf/robotiq_hande_gripper.ros2_control.xacro"/>
   <xacro:include filename="$(find robotiq_hande_description)/urdf/cylinder_inertial.xacro"/>
-  <xacro:macro name="robotiq_hande_gripper" params="name prefix parent grip_pos_min grip_pos_max tty baudrate parity data_bits stop_bit slave_id use_fake_hardware coupler_mass:=0.119">
+  <xacro:macro
+    name="robotiq_hande_gripper"
+    params="name
+            prefix
+            parent
+            grip_pos_min
+            grip_pos_max
+            tty
+            baudrate
+            parity
+            data_bits
+            stop_bit
+            slave_id
+            use_fake_hardware
+            coupler_mass:=0.119
+            xyz:='0 0 0'
+            rpy:='0 0 0'"
+  >
     <!-- ros2_control parameters  -->
     <xacro:robotiq_hande_ros2_control
@@ -32,5 +49,5 @@
     <xacro:arg name="hande_radius" default="0.0375"/>
     <joint name="${prefix}robotiq_hande_coupler_joint" type="fixed">
-      <origin xyz="0 0 0" rpy="0 0 0"/>
+      <origin xyz="${xyz}" rpy="${rpy}"/>
       <parent link="${parent}"/>
       <child link="${prefix}robotiq_hande_coupler"/>
@@ -39,5 +56,5 @@
       <visual>
         <geometry>
-          <mesh filename="package://robotiq_hande_description/meshes/io_coupler.dae"/>
+          <mesh filename="file://$(find robotiq_hande_description)/meshes/io_coupler.dae"/>
         </geometry>
       </visual>
@@ -61,5 +78,5 @@
         <origin xyz="0 0 0" rpy="0 0 0"/>
         <geometry>
-          <mesh filename="package://robotiq_hande_description/meshes/hande.dae" scale="1.0 1.0 1.0"/>
+          <mesh filename="file://$(find robotiq_hande_description)/meshes/hande.dae" scale="1.0 1.0 1.0"/>
         </geometry>
       </visual>
@@ -79,5 +96,7 @@
       <child link="${prefix}robotiq_hande_left_finger"/>
       <axis xyz="1 0 0"/>
-      <limit effort="130" lower="${grip_pos_min}" upper="${grip_pos_max}" velocity="0.15"/>
+      <limit effort="100" lower="${grip_pos_min}" upper="${grip_pos_max}" velocity="0.1"/>
+      <dynamics damping="0.5" friction="0.1"/>
+      <initial_position>0.02</initial_position>
     </joint>
     <link name="${prefix}robotiq_hande_left_finger">
@@ -85,5 +104,5 @@
         <origin xyz="0 0 0" rpy="0 0 0"/>
         <geometry>
-          <mesh filename="package://robotiq_hande_description/meshes/finger.dae" scale="1.0 1.0 1.0"/>
+          <mesh filename="file://$(find robotiq_hande_description)/meshes/finger.dae" scale="1.0 1.0 1.0"/>
         </geometry>
       </visual>
@@ -91,5 +110,5 @@
         <origin xyz="0 0 0" rpy="0 0 0"/>
         <geometry>
-          <mesh filename="package://robotiq_hande_description/meshes/finger_collision.dae" scale="1.0 1.0 1.0"/>
+          <mesh filename="file://$(find robotiq_hande_description)/meshes/finger_collision.dae" scale="1.0 1.0 1.0"/>
         </geometry>
       </collision>
@@ -105,5 +124,5 @@
       <child link="${prefix}robotiq_hande_right_finger"/>
       <axis xyz="-1 0 0"/>
-      <limit effort="130" lower="${grip_pos_min}" upper="${grip_pos_max}" velocity="0.15"/>
+      <limit effort="100" lower="${grip_pos_min}" upper="${grip_pos_max}" velocity="0.1"/>
       <mimic joint="${prefix}robotiq_hande_left_finger_joint" multiplier="1" offset="0"/>
     </joint>
@@ -112,5 +131,5 @@
         <origin xyz="0 0 0" rpy="0 0 ${pi}"/>
         <geometry>
-          <mesh filename="package://robotiq_hande_description/meshes/finger.dae" scale="1.0 1.0 1.0"/>
+          <mesh filename="file://$(find robotiq_hande_description)/meshes/finger.dae" scale="1.0 1.0 1.0"/>
         </geometry>
       </visual>
@@ -118,5 +137,5 @@
         <origin xyz="0 0 0" rpy="0 0 ${pi}"/>
         <geometry>
-          <mesh filename="package://robotiq_hande_description/meshes/finger_collision.dae" scale="1.0 1.0 1.0"/>
+          <mesh filename="file://$(find robotiq_hande_description)/meshes/finger_collision.dae" scale="1.0 1.0 1.0"/>
         </geometry>
       </collision>

File: src/ur3e_hande/ur3e_hande_description/urdf/ur3e_hande.urdf.xacro (robot description, xacro)
@@ -1,10 +1,176 @@
 <?xml version="1.0"?>
 <robot xmlns:xacro="http://www.ros.org/wiki/xacro" name="ur3e_hande">
-  <xacro:include filename="$(find robotiq_hande_description)/urdf/hande.urdf.xacro"/>
-  <xacro:include filename="$(find ur3e_description)/urdf/ur3e.urdf.xacro"/>
-  <joint name="ur3e_hande_joint" type="fixed">
-    <origin rpy="0 0 0" xyz="0 0 0"/>
-    <parent link="tool0"/>
-    <child link="robotiq_hande_coupler"/>
+  <!-- ros2 control -->
+  <xacro:include filename="$(find ur3e_hande_description)/urdf/ur3e_hande.ros2_control.xacro"/>
+  <!-- camera -->
+  <xacro:include filename="$(find ur3e_hande_description)/urdf/sensors/camera.urdf.xacro"/>
+  <!-- UR3e -->
+  <xacro:include filename="$(find ur3e_hande_description)/urdf/ur3e.urdf.xacro"/>
+    <!-- Hand-E -->
+  <xacro:include filename="$(find robotiq_hande_description)/urdf/robotiq_hande_gripper.xacro"/>
+  <!-- Table -->
+  <xacro:include filename="$(find ur3e_hande_description)/urdf/table.urdf.xacro"/>
+    <!-- include urdf for the camera mount -->
+  <xacro:include filename="$(find ur3e_hande_description)/urdf/side_extrusion_20.urdf"/>
+  <!-- insert hand-e using the macro -->
+  <xacro:robotiq_hande_gripper
+    name="robotiq_hande"
+    prefix="gripper_"
+    parent="tool0"
+    grip_pos_min="0.0"
+    grip_pos_max="0.025"
+    tty="/dev/ttyUSB0"
+    baudrate="115200"
+    parity="0"
+    data_bits="8"
+    stop_bit="1"
+    slave_id="9"
+    use_fake_hardware="true"
+  />
+  <joint name="ur3e_table_joint" type="fixed">
+    <parent link="base_link"/>
+    <child link="table"/>
+    <origin xyz="0 0 -0" rpy="0 0 0"/>
   </joint>
+  <!-- joint between the table and side extrusion -->
+  <joint name="side_extrusion_table_joint" type="fixed">
+      <parent link="table"/>
+      <child link="side_extrusion_20"/>
+      <origin rpy="0 0 0" xyz="0 0 0"/>
+  </joint>
+  <!-- Joint between camera and side extrusion -->
+  <joint name="camera_joint" type="fixed">
+    <parent link="side_extrusion_20" />
+    <child link="camera_bottom_screw_frame" />
+    <origin rpy="2.03 0.0 1.57" xyz="-0.5562625 0.542925 0.30"/>
+  </joint>
+  <!-- ROS 2 control -->
+  <xacro:ros2_control_ur3e_arm />
+  <xacro:ros2_control_hande_gripper />
+  <!-- Gazebo Sim plugin for RGB camera -->
+  <gazebo>
+      <plugin filename="gz-sim-sensors-system" name="gz::sim::systems::Sensors">
+        <render_engine>ogre2</render_engine>
+      </plugin>
+  </gazebo>
+  <gazebo reference="camera_optical_link">
+      <sensor name="camera" type="rgbd_camera">
+        <frame_id>camera_depth_optical_frame</frame_id>
+        <camera>
+         <optical_frame_id>camera_optical_link</optical_frame_id>
+          <horizontal_fov>1.5707963267948966</horizontal_fov>
+          <image>
+            <width>1280</width>
+            <height>720</height>
+            <format>RGB_INT8</format>
+          </image>
+          <clip>
+            <near>0.1</near>
+            <far>100.0</far>
+          </clip>
+          <depth_camera>
+          <optical_frame_id>camera_depth_optical_frame</optical_frame_id>
+            <clip>
+              <near>0.1</near>
+              <far>100.0</far>
+            </clip>
+          </depth_camera>
+          <distortion>
+            <k1>0.0</k1>
+            <k2>0.0</k2>
+            <k3>0.0</k3>
+            <p1>0.0</p1>
+            <p2>0.0</p2>
+            <center>0.5 0.5</center>
+          </distortion>
+          <lens>
+            <intrinsics>
+              <fx>642.312133789062</fx>
+              <fy>642.312133789062</fy>
+              <cx>636.720153808594</cx>
+              <cy>370.6181640625</cy>
+              <s>0</s>
+            </intrinsics>
+          </lens>
+          <noise>
+            <type>gaussian</type>
+            <mean>0</mean>
+            <stddev>0.007</stddev>
+          </noise>
+        </camera>
+        <always_on>1</always_on>
+        <update_rate>5</update_rate>
+        <visualize>false</visualize>
+        <topic>rgbd_camera</topic>
+        <enable_metrics>true</enable_metrics>
+      </sensor>
+  </gazebo>
+  <!-- <gazebo>
+    <plugin filename="gz-sim-joint-state-publisher-system" name="gz::sim::systems::JointStatePublisher">
+        <joint_name>shoulder_pan_joint</joint_name>
+        <joint_name>shoulder_lift_joint</joint_name>
+        <joint_name>elbow_joint</joint_name>
+        <joint_name>wrist_1_joint</joint_name>
+        <joint_name>wrist_2_joint</joint_name>
+        <joint_name>wrist_3_joint</joint_name>
+        <joint_name>gripper_robotiq_hande_left_finger_joint</joint_name>
+        <topic>/joint_states</topic>
+    </plugin>
+  </gazebo> -->
+  <gazebo>
+    <plugin filename="libgz_ros2_control-system.so" name="gz_ros2_control::GazeboSimROS2ControlPlugin">
+        <parameters>$(find ur3e_hande_description)/config/controllers_sim.yaml</parameters>
+    </plugin>
+  </gazebo>
+  <gazebo reference="table">
+    <self_collide>1</self_collide>
+    <minDepth>0.01</minDepth>
+    <mu1>1.0</mu1>
+    <mu2>1.0</mu2>
+    <restitution_coefficient>0.0</restitution_coefficient>
+    <bounce_threshold>0.0</bounce_threshold>
+  </gazebo>
+  <gazebo reference="shoulder_link">
+    <self_collide>1</self_collide>
+    <minDepth>0.01</minDepth>
+    <mu1>1.0</mu1>
+    <mu2>1.0</mu2>
+    <restitution_coefficient>0.0</restitution_coefficient>
+    <bounce_threshold>0.0</bounce_threshold>
+  </gazebo>
+  <gazebo reference="upper_arm_link">
+    <self_collide>1</self_collide>
+    <mu1>1.0</mu1>
+    <mu2>1.0</mu2>
+    <restitution_coefficient>0.0</restitution_coefficient>
+    <bounce_threshold>0.0</bounce_threshold>
+  </gazebo>
+  <gazebo reference="forearm_link">
+    <self_collide>1</self_collide>
+    <mu1>1.0</mu1>
+    <mu2>1.0</mu2>
+    <restitution_coefficient>0.0</restitution_coefficient>
+    <bounce_threshold>0.0</bounce_threshold>
+  </gazebo>
+  <gazebo reference="wrist_1_link">
+    <self_collide>1</self_collide>
+    <mu1>1.0</mu1>
+    <mu2>1.0</mu2>
+    <restitution_coefficient>0.0</restitution_coefficient>
+    <bounce_threshold>0.0</bounce_threshold>
+  </gazebo>
+  <gazebo reference="wrist_2_link">
+    <self_collide>1</self_collide>
+    <mu1>1.0</mu1>
+    <mu2>1.0</mu2>
+    <restitution_coefficient>0.0</restitution_coefficient>
+    <bounce_threshold>0.0</bounce_threshold>
+  </gazebo>
+  <gazebo reference="wrist_3_link">
+    <self_collide>1</self_collide>
+    <mu1>1.0</mu1>
+    <mu2>1.0</mu2>
+    <restitution_coefficient>0.0</restitution_coefficient>
+    <bounce_threshold>0.0</bounce_threshold>
+  </gazebo>
 </robot>

Commit message: plane+seg

File: src/hand_e/RobotiqHandeROS2Driver/robotiq_hande_description/urdf/robotiq_hande_gripper.ros2_control.xacro (robot description, xacro)
@@ -5,5 +5,5 @@
       <hardware>
         <xacro:if value="${use_fake_hardware}">
-          <plugin>gz_ros2_control/GazeboSimSystem</plugin>
+          <plugin>fake_components/GenericSystem</plugin>
         </xacro:if>
         <xacro:unless value="${use_fake_hardware}">

File: src/ur3e_hande/ur3e_hande_description/urdf/ur3e_hande.ros2_control.xacro (robot description, xacro)
@@ -92,5 +92,5 @@
         <state_interface name="effort"/>
       </joint>
-       <joint name="gripper_robotiq_hande_right_finger_joint" mimic="true">
+      <joint name="gripper_robotiq_hande_right_finger_joint">
         <state_interface name="position"/>
         <state_interface name="velocity"/>
