Commit message: hwbringup

File: src/hand_e/robotiq_hande_description/urdf/hande.urdf.xacro (robot description, xacro)
@@ -8,10 +8,10 @@
     <visual>
       <geometry>
-        <mesh filename="package://robotiq_hande_description/meshes/io_coupler.dae"/>
+        <mesh filename="file://$(find robotiq_hande_description)/meshes/io_coupler.dae"/>
       </geometry>
     </visual>
     <collision>
       <geometry>
-        <mesh filename="package://robotiq_hande_description/meshes/io_coupler.dae"/>
+        <mesh filename="file://$(find robotiq_hande_description)/meshes/io_coupler.dae"/>
       </geometry>
     </collision>
@@ -25,10 +25,10 @@
     <visual>
       <geometry>
-        <mesh filename="package://robotiq_hande_description/meshes/hande.dae" scale="1.0 1.0 1.0"/>
+        <mesh filename="file://$(find robotiq_hande_description)/meshes/hande.dae" scale="1.0 1.0 1.0"/>
       </geometry>
     </visual>
     <collision>
       <geometry>
-        <mesh filename="package://robotiq_hande_description/meshes/hande.dae" scale="1.0 1.0 1.0"/>
+        <mesh filename="file://$(find robotiq_hande_description)/meshes/hande.dae" scale="1.0 1.0 1.0"/>
       </geometry>
     </collision>
@@ -44,10 +44,10 @@
     <visual>
       <geometry>
-        <mesh filename="package://robotiq_hande_description/meshes/finger.dae" scale="1.0 1.0 1.0"/>
+        <mesh filename="file://$(find robotiq_hande_description)/meshes/finger.dae" scale="1.0 1.0 1.0"/>
       </geometry>
     </visual>
     <collision>
       <geometry>
-        <mesh filename="package://robotiq_hande_description/meshes/finger_collision.dae" scale="1.0 1.0 1.0"/>
+        <mesh filename="file://$(find robotiq_hande_description)/meshes/finger_collision.dae" scale="1.0 1.0 1.0"/>
       </geometry>
     </collision>
@@ -65,5 +65,5 @@
       <origin rpy="0 0 3.14159"/>
       <geometry>
-        <mesh filename="package://robotiq_hande_description/meshes/finger.dae" scale="1.0 1.0 1.0"/>
+        <mesh filename="file://$(find robotiq_hande_description)/meshes/finger.dae" scale="1.0 1.0 1.0"/>
       </geometry>
     </visual>
@@ -71,5 +71,5 @@
       <origin rpy="0 0 3.14159"/>
       <geometry>
-        <mesh filename="package://robotiq_hande_description/meshes/finger_collision.dae" scale="1.0 1.0 1.0"/>
+        <mesh filename="file://$(find robotiq_hande_description)/meshes/finger_collision.dae" scale="1.0 1.0 1.0"/>
       </geometry>
     </collision>

File: src/hand_e/robotiq_hande_description/urdf_hw/robotiq_hande_gripper.urdf.xacro (robot description, xacro)
@@ -16,5 +16,5 @@
   <xacro:arg name="use_fake_hardware" default="true"/>
   <xacro:include filename="$(find robotiq_hande_description)/urdf_hw/robotiq_hande_gripper.xacro"/>
-  <link name="$(arg parent)"/>
+  <!-- <link name="$(arg parent)"/> -->
   <xacro:robotiq_hande_gripper
     name="robotiq_hande_gripper"

File: src/hand_e/robotiq_hande_description/urdf_hw/robotiq_hande_gripper.xacro (robot description, xacro)
@@ -64,5 +64,5 @@
       <visual>
         <geometry>
-          <mesh filename="package://robotiq_hande_description/meshes/io_coupler.dae"/>
+          <mesh filename="file://$(find robotiq_hande_description)/meshes/io_coupler.dae"/>
         </geometry>
       </visual>
@@ -86,5 +86,5 @@
         <origin xyz="0 0 0" rpy="0 0 0"/>
         <geometry>
-          <mesh filename="package://robotiq_hande_description/meshes/hande.dae" scale="1.0 1.0 1.0"/>
+          <mesh filename="file://$(find robotiq_hande_description)/meshes/hande.dae" scale="1.0 1.0 1.0"/>
         </geometry>
       </visual>
@@ -110,5 +110,5 @@
         <origin xyz="0 0 0" rpy="0 0 0"/>
         <geometry>
-          <mesh filename="package://robotiq_hande_description/meshes/finger.dae" scale="1.0 1.0 1.0"/>
+          <mesh filename="file://$(find robotiq_hande_description)/meshes/finger.dae" scale="1.0 1.0 1.0"/>
         </geometry>
       </visual>
@@ -116,5 +116,5 @@
         <origin xyz="0 0 0" rpy="0 0 0"/>
         <geometry>
-          <mesh filename="package://robotiq_hande_description/meshes/finger_collision.dae" scale="1.0 1.0 1.0"/>
+          <mesh filename="file://$(find robotiq_hande_description)/meshes/finger_collision.dae" scale="1.0 1.0 1.0"/>
         </geometry>
       </collision>
@@ -137,5 +137,5 @@
         <origin xyz="0 0 0" rpy="0 0 ${pi}"/>
         <geometry>
-          <mesh filename="package://robotiq_hande_description/meshes/finger.dae" scale="1.0 1.0 1.0"/>
+          <mesh filename="file://$(find robotiq_hande_description)/meshes/finger.dae" scale="1.0 1.0 1.0"/>
         </geometry>
       </visual>
@@ -143,5 +143,5 @@
         <origin xyz="0 0 0" rpy="0 0 ${pi}"/>
         <geometry>
-          <mesh filename="package://robotiq_hande_description/meshes/finger_collision.dae" scale="1.0 1.0 1.0"/>
+          <mesh filename="file://$(find robotiq_hande_description)/meshes/finger_collision.dae" scale="1.0 1.0 1.0"/>
         </geometry>
       </collision>

File: src/ur3e_hande/ur3e_hande_description/urdf/ur3e_hande_hw.urdf.xacro (robot description, xacro)
@@ -15,8 +15,7 @@
   <xacro:arg name="slave_id" default="9"/>
   <xacro:arg name="frequency_hz" default="10"/>
-  <xacro:arg name="create_socat_tty" default="false"/>
+  <xacro:arg name="create_socat_tty" default="true"/>
   <xacro:arg name="socat_ip_address" default="192.168.77.22"/>
   <xacro:arg name="socat_port" default="54321"/>
-  <xacro:arg name="use_fake_hardware" default="true"/>
   <xacro:arg name="import_ur3e" default="true"/>
   <xacro:arg name="import_hande" default="true"/>
@@ -27,5 +26,5 @@
     <!-- Import hande xacro -->
   <xacro:if value="$(arg import_hande)">
-    <xacro:include filename="$(find robotiq_hande_description)/urdf_hw/robotiq_hande_gripper.urdf.xacro"/>
+    <xacro:include filename="$(find robotiq_hande_description)/urdf_hw/robotiq_hande_gripper.xacro"/>
   </xacro:if>
    <!-- import main macro -->
@@ -63,4 +62,6 @@
    <xacro:arg name="tool_device_name" default="/tmp/ttyUR" />
    <xacro:arg name="tool_tcp_port" default="54321" />
+   <!--When using gazebo simulations absolute paths are necessary.-->
+   <xacro:arg name="force_abs_paths" default="true" />
      <!-- Simulation parameters -->
    <xacro:arg name="use_fake_hardware" default="false" />
@@ -73,4 +74,6 @@
    <!-- convert to property to use substitution in function -->
    <xacro:property name="initial_positions_file" default="$(arg initial_positions_file)"/>
+   <!-- realsense loc: left or right of robot base frame -->
+   <xacro:arg name="cam_loc" default="right"/>
    <!-- create link fixed to the "world" -->
    <link name="world" />
@@ -78,38 +81,18 @@
   <xacro:if value="$(arg import_ur3e)">
     <xacro:ur_robot
-      name="$(arg name)"
-      tf_prefix="$(arg tf_prefix)"
-      parent="world"
-      joint_limits_parameters_file="$(arg joint_limit_params)"
-      kinematics_parameters_file="$(arg kinematics_params)"
-      physical_parameters_file="$(arg physical_params)"
-      visual_parameters_file="$(arg visual_params)"
-      safety_limits="$(arg safety_limits)"
-      safety_pos_margin="$(arg safety_pos_margin)"
-      safety_k_position="$(arg safety_k_position)"
-      use_fake_hardware="$(arg use_fake_hardware)"
-      fake_sensor_commands="$(arg fake_sensor_commands)"
-      sim_gazebo="$(arg sim_gazebo)"
-      sim_ignition="$(arg sim_ignition)"
-      headless_mode="$(arg headless_mode)"
-      initial_positions="${xacro.load_yaml(initial_positions_file)}"
-      use_tool_communication="$(arg use_tool_communication)"
-      tool_voltage="$(arg tool_voltage)"
-      tool_parity="$(arg tool_parity)"
-      tool_baud_rate="$(arg tool_baud_rate)"
-      tool_stop_bits="$(arg tool_stop_bits)"
-      tool_rx_idle_chars="$(arg tool_rx_idle_chars)"
-      tool_tx_idle_chars="$(arg tool_tx_idle_chars)"
-      tool_device_name="$(arg tool_device_name)"
-      tool_tcp_port="$(arg tool_tcp_port)"
-      robot_ip="$(arg robot_ip)"
-      script_filename="$(arg script_filename)"
-      output_recipe_filename="$(arg output_recipe_filename)"
-      input_recipe_filename="$(arg input_recipe_filename)"
-      reverse_ip="$(arg reverse_ip)"
-      script_command_port="$(arg script_command_port)"
-      >
-      <origin xyz="0 0 0" rpy="0 0 0" />          <!-- position robot in the world -->
-    </xacro:ur_robot>
+     name="$(arg name)"
+     tf_prefix="$(arg tf_prefix)"
+     parent="world"
+     joint_limits_parameters_file="$(arg joint_limit_params)"
+     kinematics_parameters_file="$(arg kinematics_params)"
+     physical_parameters_file="$(arg physical_params)"
+     visual_parameters_file="$(arg visual_params)"
+     safety_limits="$(arg safety_limits)"
+     safety_pos_margin="$(arg safety_pos_margin)"
+     safety_k_position="$(arg safety_k_position)"
+     force_abs_paths="$(arg force_abs_paths)"
+     >
+     <origin xyz="0 0 0.85" rpy="0 0 0" />          <!-- position robot in the world -->
+   </xacro:ur_robot>
    </xacro:if>
     <xacro:if value="$(arg import_hande)">
@@ -134,5 +117,5 @@
     </xacro:if>
   <!-- Import table -->
-  <xacro:include filename="$(find ur3e_description)/urdf/table.urdf"/>
+  <xacro:include filename="$(find ur3e_hande_description)/urdf/table.urdf.xacro"/>
   <!-- Import realsense -->
   <xacro:if value="${is_import_ur3e and is_import_camera}">
@@ -140,7 +123,10 @@
   </xacro:if>
   <!-- Use the sensor_d435i macro; this is the camera on the right; add a unique namespace (e.g. camera2) if using both cameras-->
+  <!-- Need to make a parameter -->
   <xacro:if value="${is_import_ur3e and is_import_camera}">
     <xacro:sensor_d435i parent="world">
-        <origin rpy="0.0 0.698131 0" xyz="-0.522625 0.542925 0.3683"/>
+        <origin rpy="0.0 0.698131 -180" xyz="0.522625 0.542925 0.3683"/>
+        <!-- use this for cam_loc:=left -->
+        <!-- <origin rpy="0.0 0.698131 0" xyz="-0.522625 0.542925 0.3683"/>   -->
     </xacro:sensor_d435i>
   </xacro:if>
