Commit message: hw lab

File: src/hand_e/robotiq_hande_description/urdf/robotiq_hande_gripper.ros2_control.xacro (robot description, xacro)
@@ -10,20 +10,4 @@
           <plugin>mock_components/GenericSystem</plugin>
         </xacro:if>
-        <xacro:unless value="${use_fake_hardware}">
-          <plugin>robotiq_hande_driver/RobotiqHandeHardwareInterface</plugin>
-          <param name="grip_pos_min">${grip_pos_min}</param>
-          <param name="grip_pos_max">${grip_pos_max}</param>
-          <param name="tty_port">${tty_port}</param>
-          <param name="baudrate">${baudrate}</param>
-          <param name="parity">${parity}</param>
-          <param name="data_bits">${data_bits}</param>
-          <param name="stop_bit">${stop_bit}</param>
-          <param name="slave_id">${slave_id}</param>
-          <param name="frequency_hz">${frequency_hz}</param>
-          <param name="create_socat_tty">${create_socat_tty}</param>
-          <param name="socat_ip_address">${socat_ip_address}</param>
-          <param name="socat_port">${socat_port}</param>
-        </xacro:unless>
-      </hardware>
       <!-- The right finger joint uses the mimic feature -->
       <joint name="${prefix}robotiq_hande_left_finger_joint">

File: src/ur3e/ur3e_description/urdf/ur3e.urdf.xacro (robot description, xacro)
@@ -14,4 +14,5 @@
   <xacro:arg name="extrusion_y" default="0.533"/>
   <xacro:arg name="extrusion_z" default="0.50"/>
+  <xacro:arg name="extrusion_width" default="0.04"/>
   <xacro:arg name="extrusion_roll" default="0.0"/>
   <xacro:arg name="extrusion_pitch" default="0.0"/>
@@ -19,14 +20,23 @@
   <xacro:arg name="cam_offset_x" default="0.002"/>
   <xacro:arg name="cam_offset_y" default="0.0"/>
-  <xacro:arg name="cam_offset_z" default="0.0105"/>
-  <xacro:arg name="cam_roll" default="0.0"/>
-  <xacro:arg name="cam_pitch" default="0.32"/>
-  <xacro:arg name="cam_yaw" default="-3.14"/>
+  <xacro:arg name="cam_offset_z" default="0.0"/>
+    <xacro:arg name="camera_x" default="0.0"/>
+  <xacro:arg name="camera_y" default="0.0"/>
+  <xacro:arg name="mount_height" default="0.467"/>
+  <xacro:arg name="camera_roll" default="0.0"/>
+  <xacro:arg name="camera_pitch" default="0.32"/>
+  <xacro:arg name="camera_yaw" default="-3.14"/>
+  <xacro:arg name="realsense_width" default="0.09"/>
+  <xacro:arg name="realsense_depth" default="0.025"/>
+  <xacro:arg name="realsense_height" default="0.025"/>
   <xacro:property name="cam_offset_x" value="$(arg cam_offset_x)"/>
   <xacro:property name="cam_offset_y" value="$(arg cam_offset_y)"/>
   <xacro:property name="cam_offset_z" value="$(arg cam_offset_z)"/>
-  <xacro:property name="cam_roll" value="$(arg cam_roll)"/>
-  <xacro:property name="cam_pitch" value="$(arg cam_pitch)"/>
-  <xacro:property name="cam_yaw" value="$(arg cam_yaw)"/>
+  <xacro:property name="camera_x" value="$(arg camera_x)"/>
+  <xacro:property name="camera_y" value="$(arg camera_y)"/>
+  <xacro:property name="mount_height" value="$(arg mount_height)"/>
+  <xacro:property name="camera_roll" value="$(arg camera_roll)"/>
+  <xacro:property name="camera_pitch" value="$(arg camera_pitch)"/>
+  <xacro:property name="camera_yaw" value="$(arg camera_yaw)"/>
   <xacro:property name="extrusion_x" value="$(arg extrusion_x)"/>
   <xacro:property name="extrusion_y" value="$(arg extrusion_y)"/>
@@ -35,4 +45,5 @@
   <xacro:property name="extrusion_pitch" value="$(arg extrusion_pitch)"/>
   <xacro:property name="extrusion_yaw" value="$(arg extrusion_yaw)"/>
+  <xacro:property name="extrusion_width" value="$(arg extrusion_width)"/>
    <!-- parameters -->
    <xacro:arg name="tf_prefix" default="" />
@@ -192,18 +203,41 @@
   </xacro:sensor_d435i> -->
   <!-- Use the sensor_d435i macro; this is the camera on the right; add a unique namespace (e.g. camera2) if using both cameras-->
- <!-- <xacro:sensor_d435i parent="side_extrusion_20">
+ <xacro:sensor_d435i parent="table" use_nominal_extrinsics="true" add_plug="true" use_mesh="true" publish_pointcloud="true">
       <origin
-      xyz="${cam_offset_x} ${cam_offset_y} ${cam_offset_z}"
-      rpy="${cam_roll} ${cam_pitch} ${cam_yaw}"
+      xyz="${cam_offset_x} ${cam_offset_y} ${mount_height}"
+      rpy="${camera_roll} ${camera_pitch} ${camera_yaw}"
       />
+  </xacro:sensor_d435i>
+  <!-- <xacro:sensor_d435i parent="table" use_nominal_extrinsics="true" add_plug="true" use_mesh="true" publish_pointcloud="true">
+      <origin rpy="0.0 0.5 -3.14" xyz="0.555 0.5333 0.467"/>
   </xacro:sensor_d435i> -->
-  <xacro:sensor_d435i parent="base_link">
-        <origin rpy="0.0 0.5 -3.14" xyz="0.555 0.5333 0.467"/>
-    </xacro:sensor_d435i>
-  <link name="camera_optical_link"/>
+  <!-- <link name="camera_optical_link"/>
   <joint name="align_camera_joint" type="fixed">
     <parent link="camera_link"/>
     <child link="camera_optical_link"/>
-    <origin xyz="0 0 0" rpy="${-pi/2} 0 ${pi}"/> <!-- sim: -3.14 -1.57 1.57; recc: ${-pi/2} 0 ${-pi/2}-->
-  </joint>
+    <origin xyz="0 0 0" rpy="${-pi/2} 0 ${pi}"/>
+  </joint> -->
+<!-- sim: -3.14 -1.57 1.57; recc: ${-pi/2} 0 ${-pi/2}-->
+<link name="back_wall">
+  <visual>
+    <origin xyz="-0.13 0.0 0.50" rpy="0 0 0"/>
+    <geometry>
+      <box size="0.05 1.5 1.0"/> <!-- thickness, width, height -->
+    </geometry>
+    <material name="gray">
+      <color rgba="0.6 0.6 0.6 1.0"/>
+    </material>
+  </visual>
+  <collision>
+    <origin xyz="-0.13 0.0 0.50" rpy="0 0 0"/>
+    <geometry>
+      <box size="0.05 1.5 1.0"/>
+    </geometry>
+  </collision>
+</link>
+<joint name="back_wall_fixed" type="fixed">
+  <parent link="base_link"/>
+  <child link="back_wall"/>
+  <origin xyz="0 0 0" rpy="0 0 0"/>
+</joint>
 </robot>

File: src/ur3e_hande/ur3e_hande_description/urdf/ur3e_hande_hw.urdf.xacro (robot description, xacro)
@@ -158,5 +158,5 @@
       <origin rpy="0.0 0.4712 1.57" xyz="0.381 -0.125 0.415925"/>
   </xacro:sensor_d435i> -->
-  <!-- Use the sensor_d435i macro; this is the camera on the right; add a unique namespace (e.g. camera2) if using both cameras-->
+  <!-- Use the sensor_d435i macro; this is the camera on the right/left; add a unique namespace (e.g. camera2) if using multiple cameras-->
   <xacro:if value="${is_import_ur3e and is_import_camera}">
     <xacro:sensor_d435i parent="world">

File: src/ur3e_hande/ur3e_hande_moveit_config/config/ur3e_hande.srdf.xacro (robot description, xacro)
@@ -55,5 +55,5 @@
     <joint name="robotiq_hande_right_finger_joint" value="0"/>
   </group_state>
-  <!--END EFFECTOR: Purpose: Represent information about an end effector.-->
+  <!--END EFFECTOR: Purpose: Represents information about an end effector.-->
   <end_effector group="gripper" name="hand_ee" parent_group="ur_manipulator" parent_link="wrist_3_link"/>
   <!--DISABLE COLLISIONS: By default it is assumed that any link of the robot could potentially come into collision with any other link in the robot. This tag disables collision checking between a specified pair of links. -->

File: src/ur3e_hande/ur3e_hande_moveit_config/config/ur3e_hande.urdf.xacro (robot description, xacro)
@@ -38,5 +38,3 @@
       use_fake_hardware="${use_fake_hardware}"
     />
-    <!-- HW interface in the works; NA for now -->
-    <!-- <xacro:ur3e_hande_ros2_control name="robotiq_hande_controllers/RobotiqHandeHardwareInterface" initial_positions_file="$(arg initial_positions_file)"/> -->
 </robot>

Commit message: cleanup

File: src/hand_e/robotiq_hande_description/urdf/robotiq_hande_gripper.ros2_control.xacro (robot description, xacro)
@@ -10,4 +10,5 @@
           <plugin>mock_components/GenericSystem</plugin>
         </xacro:if>
+      </hardware>
       <!-- The right finger joint uses the mimic feature -->
       <joint name="${prefix}robotiq_hande_left_finger_joint">

File: src/ur3e/ur3e_description/urdf/ur3e.urdf.xacro (robot description, xacro)
@@ -177,5 +177,5 @@
   </xacro:if>
   <!-- Import table -->
-   <xacro:include filename="$(find ur3e_description)/urdf/table.urdf"/>
+   <xacro:include filename="$(find ur3e_description)/urdf/table.urdf.xacro"/>
   <!-- Joint between table and ur -->
   <joint name="table_joint" type="fixed">
@@ -203,5 +203,5 @@
   </xacro:sensor_d435i> -->
   <!-- Use the sensor_d435i macro; this is the camera on the right; add a unique namespace (e.g. camera2) if using both cameras-->
- <xacro:sensor_d435i parent="table" use_nominal_extrinsics="true" add_plug="true" use_mesh="true" publish_pointcloud="true">
+ <xacro:sensor_d435i parent="table" use_nominal_extrinsics="true">
       <origin
       xyz="${extrusion_x} ${extrusion_y} ${mount_height}"
@@ -239,5 +239,5 @@
   <parent link="base_link"/>
   <child link="back_wall"/>
-  <origin xyz="0 0 0" rpy="0 0 0"/>
+  <origin xyz="0 0 0" rpy="0 0 1.57"/>
 </joint>
 </robot>
