Commit message: docker-lab

File: src/ur3e_hande/ur3e_hande_description/urdf/ur3e_hande_hw.urdf.xacro (robot description, xacro)
@@ -8,5 +8,5 @@
   <xacro:arg name="grip_pos_min" default="0"/>
   <xacro:arg name="grip_pos_max" default="0.025"/>
-  <xacro:arg name="tty" default="/tmp/ttyUR"/>
+  <xacro:arg name="tty_port" default="/tmp/ttyUR"/>
   <xacro:arg name="baudrate" default="115200"/>
   <xacro:arg name="parity" default="N"/>
@@ -14,5 +14,9 @@
   <xacro:arg name="stop_bit" default="1"/>
   <xacro:arg name="slave_id" default="9"/>
-  <xacro:arg name="use_fake_hardware" default="false"/>
+  <xacro:arg name="frequency_hz" default="10"/>
+  <xacro:arg name="create_socat_tty" default="false"/>
+  <xacro:arg name="socat_ip_address" default="192.168.77.22"/>
+  <xacro:arg name="socat_port" default="54321"/>
+  <xacro:arg name="use_fake_hardware" default="true"/>
   <xacro:arg name="import_ur3e" default="true"/>
   <xacro:arg name="import_hande" default="true"/>
@@ -23,5 +27,5 @@
     <!-- Import hande xacro -->
   <xacro:if value="$(arg import_hande)">
-    <xacro:include filename="$(find robotiq_hande_description)/urdf/robotiq_hande_gripper.urdf.xacro"/>
+    <xacro:include filename="$(find robotiq_hande_description)/urdf_hw/robotiq_hande_gripper.urdf.xacro"/>
   </xacro:if>
    <!-- import main macro -->
@@ -50,5 +54,5 @@
    <xacro:arg name="script_command_port" default="50004"/>
    <!--   tool communication related parameters-->
-   <xacro:arg name="use_tool_communication" default="true" />
+   <xacro:arg name="use_tool_communication" default="false" />
    <xacro:arg name="tool_voltage" default="24" />
    <xacro:arg name="tool_parity" default="N" />
@@ -109,6 +113,6 @@
     </xacro:ur_robot>
    </xacro:if>
-    <!-- <xacro:if value="$(arg import_hande)"> -->
-      <!-- <xacro:robotiq_hande_gripper
+    <xacro:if value="$(arg import_hande)">
+      <xacro:robotiq_hande_gripper
         name="$(arg hande_name)"
         prefix=""
@@ -116,5 +120,5 @@
         grip_pos_min="$(arg grip_pos_min)"
         grip_pos_max="$(arg grip_pos_max)"
-        tty="$(arg tty)"
+        tty_port="$(arg tty_port)"
         baudrate="$(arg baudrate)"
         parity="$(arg parity)"
@@ -122,28 +126,11 @@
         stop_bit="$(arg stop_bit)"
         slave_id="$(arg slave_id)"
+        frequency_hz="$(arg frequency_hz)"
+        create_socat_tty="$(arg create_socat_tty)"
+        socat_ip_address="$(arg socat_ip_address)"
+        socat_port="$(arg socat_port)"
         use_fake_hardware="$(arg use_fake_hardware)"
-      /> -->
-    <!-- </xacro:if> -->
-   <xacro:if value="$(arg sim_gazebo)">
-    <!-- Gazebo plugins -->
-    <gazebo reference="world">
-    </gazebo>
-    <gazebo>
-      <plugin filename="libgazebo_ros2_control.so" name="gazebo_ros2_control">
-        <parameters>$(arg simulation_controllers)</parameters>
-      </plugin>
-    </gazebo>
-  </xacro:if>
-  <xacro:if value="$(arg sim_ignition)">
-    <!-- Gazebo plugins -->
-    <gazebo reference="world">
-    </gazebo>
-    <gazebo>
-      <plugin filename="libign_ros2_control-system.so" name="ign_ros2_control::IgnitionROS2ControlPlugin">
-        <parameters>$(arg simulation_controllers)</parameters>
-        <controller_manager_node_name>$(arg tf_prefix)controller_manager</controller_manager_node_name>
-      </plugin>
-    </gazebo>
-  </xacro:if>
+      />
+    </xacro:if>
   <!-- Import table -->
   <xacro:include filename="$(find ur3e_description)/urdf/table.urdf"/>
@@ -152,8 +139,4 @@
     <xacro:include filename="$(find realsense2_description)/urdf/_d435i.urdf.xacro"/>
   </xacro:if>
-  <!-- Use the sensor_d435i macro with a unique name (camera_top)-->
-  <!-- <xacro:sensor_d435i parent="world" name="camera1">
-      <origin rpy="0.0 0.4712 1.57" xyz="0.381 -0.125 0.415925"/>
-  </xacro:sensor_d435i> -->
   <!-- Use the sensor_d435i macro; this is the camera on the right; add a unique namespace (e.g. camera2) if using both cameras-->
   <xacro:if value="${is_import_ur3e and is_import_camera}">
@@ -171,5 +154,5 @@
   </xacro:if>
   <!-- Joint between ur3e and hande -->
-<xacro:if value="${is_import_ur3e and is_import_hande}">
+<!-- <xacro:if value="${is_import_ur3e and is_import_hande}">
   <joint name="ur3e_hande_joint" type="fixed">
     <origin rpy="${pi/2} ${-pi/2} 0" xyz="0.00574 .03656 .01111"/>
@@ -177,4 +160,4 @@
     <child link="hande_link"/>
   </joint>
-</xacro:if>
+</xacro:if> -->
 </robot>

Commit message: updates

File: src/ur3e_hande/ur3e_hande_description/urdf/ur3e_hande_hw.urdf.xacro (robot description, xacro)
@@ -18,4 +18,5 @@
   <xacro:arg name="socat_ip_address" default="192.168.77.22"/>
   <xacro:arg name="socat_port" default="54321"/>
+  <xacro:arg name="camera_mount_frame" default="camera_mount"/>
   <xacro:arg name="import_ur3e" default="true"/>
   <xacro:arg name="import_hande" default="true"/>
@@ -38,5 +39,5 @@
    <xacro:arg name="tf_prefix" default="" />
    <xacro:arg name="joint_limit_params" default="$(find ur_description)/config/$(arg ur_type)/joint_limits.yaml"/>
-   <xacro:arg name="kinematics_params" default="$(find ur_description)/config/$(arg ur_type)/default_kinematics.yaml"/>
+   <!-- <xacro:arg name="kinematics_params" default="/home/robot/kinematic_config/ur3e_mrc.yaml"/> -->
    <xacro:arg name="physical_params" default="$(find ur_description)/config/$(arg ur_type)/physical_parameters.yaml"/>
    <xacro:arg name="visual_params" default="$(find ur_description)/config/$(arg ur_type)/visual_parameters.yaml"/>
@@ -74,6 +75,4 @@
    <!-- convert to property to use substitution in function -->
    <xacro:property name="initial_positions_file" default="$(arg initial_positions_file)"/>
-   <!-- realsense loc: left or right of robot base frame -->
-   <xacro:arg name="cam_loc" default="right"/>
    <!-- create link fixed to the "world" -->
    <link name="world" />
@@ -85,5 +84,4 @@
      parent="world"
      joint_limits_parameters_file="$(arg joint_limit_params)"
-     kinematics_parameters_file="$(arg kinematics_params)"
      physical_parameters_file="$(arg physical_params)"
      visual_parameters_file="$(arg visual_params)"
@@ -125,8 +123,7 @@
   <!-- Need to make a parameter -->
   <xacro:if value="${is_import_ur3e and is_import_camera}">
-    <xacro:sensor_d435i parent="world">
-        <origin rpy="0.0 0.698131 -180" xyz="0.522625 0.542925 0.3683"/>
-        <!-- use this for cam_loc:=left -->
-        <!-- <origin rpy="0.0 0.698131 0" xyz="-0.522625 0.542925 0.3683"/>   -->
+    <xacro:sensor_d435i parent="$(arg camera_mount_frame)">
+        <!-- <origin rpy="0.0 0.698131 -180" xyz="0.522625 0.542925 0.3683"/>   --> <!-- right camera -->
+        <!-- <origin rpy="0.0 0.698131 0" xyz="-0.522625 0.542925 0.3683"/>   --> <!-- left camera -->
     </xacro:sensor_d435i>
   </xacro:if>

Commit message: hande

File: src/ur3e_hande/ur3e_hande_description/urdf/ur3e_hande_hw.urdf.xacro (robot description, xacro)
@@ -18,5 +18,4 @@
   <xacro:arg name="socat_ip_address" default="192.168.77.22"/>
   <xacro:arg name="socat_port" default="54321"/>
-  <xacro:arg name="camera_mount_frame" default="camera_mount"/>
   <xacro:arg name="import_ur3e" default="true"/>
   <xacro:arg name="import_hande" default="true"/>
@@ -39,5 +38,5 @@
    <xacro:arg name="tf_prefix" default="" />
    <xacro:arg name="joint_limit_params" default="$(find ur_description)/config/$(arg ur_type)/joint_limits.yaml"/>
-   <!-- <xacro:arg name="kinematics_params" default="/home/robot/kinematic_config/ur3e_mrc.yaml"/> -->
+   <xacro:arg name="kinematics_params" default="/home/robot/kinematic_config/ur3e_mrc.yaml"/>
    <xacro:arg name="physical_params" default="$(find ur_description)/config/$(arg ur_type)/physical_parameters.yaml"/>
    <xacro:arg name="visual_params" default="$(find ur_description)/config/$(arg ur_type)/visual_parameters.yaml"/>
@@ -86,4 +85,5 @@
      physical_parameters_file="$(arg physical_params)"
      visual_parameters_file="$(arg visual_params)"
+     kinematics_parameters_file="$(arg kinematics_params)"
      safety_limits="$(arg safety_limits)"
      safety_pos_margin="$(arg safety_pos_margin)"
@@ -121,9 +121,8 @@
   </xacro:if>
   <!-- Use the sensor_d435i macro; this is the camera on the right; add a unique namespace (e.g. camera2) if using both cameras-->
-  <!-- Need to make a parameter -->
   <xacro:if value="${is_import_ur3e and is_import_camera}">
-    <xacro:sensor_d435i parent="$(arg camera_mount_frame)">
-        <!-- <origin rpy="0.0 0.698131 -180" xyz="0.522625 0.542925 0.3683"/>   --> <!-- right camera -->
-        <!-- <origin rpy="0.0 0.698131 0" xyz="-0.522625 0.542925 0.3683"/>   --> <!-- left camera -->
+    <xacro:sensor_d435i parent="base_link">
+      <origin rpy="0 0.52 0" xyz="-0.546 0.533 0.467"/>   <!-- right camera -->
+      <!-- <origin rpy="0.0 0.698131 0" xyz="-0.522625 0.542925 0.3683"/>   --> <!-- left camera -->
     </xacro:sensor_d435i>
   </xacro:if>
@@ -141,5 +140,5 @@
     <origin rpy="${pi/2} ${-pi/2} 0" xyz="0.00574 .03656 .01111"/>
     <parent link="tool0"/>
-    <child link="hande_link"/>
+    <child link="robotiq_hande_coupler"/>
   </joint>
 </xacro:if> -->
