Commit message: cleanup

File: src/ur3e_hande/ur3e_hande_description/urdf/ur3e.urdf.xacro (robot description, xacro)
@@ -11,5 +11,5 @@
    <xacro:arg name="tf_prefix" default="" />
    <xacro:arg name="joint_limit_params" default="$(find ur_description)/config/$(arg ur_type)/joint_limits.yaml"/>
-   <xacro:arg name="kinematics_params" default="/home/robot/kinematic_config/ur3e_mrc.yaml"/>
+   <xacro:arg name="kinematics_params" default="$(find ur3e_hande_description)/config/ur3e_mrc.yaml"/>
    <xacro:arg name="physical_params" default="$(find ur_description)/config/$(arg ur_type)/physical_parameters.yaml"/>
    <xacro:arg name="visual_params" default="$(find ur_description)/config/$(arg ur_type)/visual_parameters.yaml"/>

File: src/ur3e_hande/ur3e_hande_description/urdf/ur3e_hande.urdf.xacro (robot description, xacro)
@@ -1,4 +1,34 @@
 <?xml version="1.0"?>
 <robot xmlns:xacro="http://www.ros.org/wiki/xacro" name="ur3e_hande">
+  <!-- Required by UR macros -->
+  <xacro:arg name="name" default="ur3e"/>
+  <xacro:arg name="ur_type" default="ur3e"/>
+  <xacro:arg name="tf_prefix" default=""/>
+  <xacro:arg name="prefix" default=""/>
+  <!-- Extrusion -->
+  <xacro:arg name="extrusion_x" default="-0.5762625"/>
+  <xacro:arg name="extrusion_y" default="0.542925"/>
+  <xacro:arg name="extrusion_z" default="0.291"/>
+  <xacro:arg name="extrusion_roll" default="0.0"/>
+  <xacro:arg name="extrusion_pitch" default="0.0"/>
+  <xacro:arg name="extrusion_yaw" default="0.0"/>
+  <xacro:arg name="cam_offset_x" default="0.02"/>
+  <xacro:arg name="cam_offset_y" default="0.0"/>
+  <xacro:arg name="cam_offset_z" default="0.01"/>
+  <xacro:arg name="cam_roll" default="2.03"/>
+  <xacro:arg name="cam_pitch" default="0.0"/>
+  <xacro:arg name="cam_yaw" default="1.57"/>
+  <xacro:property name="cam_offset_x" value="$(arg cam_offset_x)"/>
+  <xacro:property name="cam_offset_y" value="$(arg cam_offset_y)"/>
+  <xacro:property name="cam_offset_z" value="$(arg cam_offset_z)"/>
+  <xacro:property name="cam_roll" value="$(arg cam_roll)"/>
+  <xacro:property name="cam_pitch" value="$(arg cam_pitch)"/>
+  <xacro:property name="cam_yaw" value="$(arg cam_yaw)"/>
+  <xacro:property name="extrusion_x" value="$(arg extrusion_x)"/>
+  <xacro:property name="extrusion_y" value="$(arg extrusion_y)"/>
+  <xacro:property name="extrusion_z" value="$(arg extrusion_z)"/>
+  <xacro:property name="extrusion_roll" value="$(arg extrusion_roll)"/>
+  <xacro:property name="extrusion_pitch" value="$(arg extrusion_pitch)"/>
+  <xacro:property name="extrusion_yaw" value="$(arg extrusion_yaw)"/>
   <!-- ros2 control -->
   <xacro:include filename="$(find ur3e_hande_description)/urdf/ur3e_hande.ros2_control.xacro"/>
@@ -12,5 +42,5 @@
   <xacro:include filename="$(find ur3e_hande_description)/urdf/table.urdf.xacro"/>
     <!-- include urdf for the camera mount -->
-  <xacro:include filename="$(find ur3e_hande_description)/urdf/side_extrusion_20.urdf"/>
+  <xacro:include filename="$(find ur3e_hande_description)/urdf/side_extrusion_20.urdf.xacro"/>
   <!-- insert hand-e using the macro -->
   <xacro:robotiq_hande_gripper
@@ -33,15 +63,21 @@
     <origin xyz="0 0 -0" rpy="0 0 0"/>
   </joint>
-  <!-- joint between the table and side extrusion -->
-  <joint name="side_extrusion_table_joint" type="fixed">
-      <parent link="table"/>
-      <child link="side_extrusion_20"/>
-      <origin rpy="0 0 0" xyz="0 0 0"/>
-  </joint>
+  <xacro:side_extrusion_20
+  parent="table"
+  x="$(arg extrusion_x)"
+  y="$(arg extrusion_y)"
+  z="$(arg extrusion_z)"
+  roll="$(arg extrusion_roll)"
+  pitch="$(arg extrusion_pitch)"
+  yaw="$(arg extrusion_yaw)"
+  />
   <!-- Joint between camera and side extrusion -->
   <joint name="camera_joint" type="fixed">
     <parent link="side_extrusion_20" />
     <child link="camera_bottom_screw_frame" />
-    <origin rpy="2.03 0.0 1.57" xyz="-0.5562625 0.542925 0.30"/>
+    <origin
+    xyz="${cam_offset_x} ${cam_offset_y} ${cam_offset_z}"
+    rpy="${cam_roll} ${cam_pitch} ${cam_yaw}"
+    />
   </joint>
   <!-- ROS 2 control -->

File: src/ur3e_hande/ur3e_hande_description/urdf/ur3e_hande_hw.urdf.xacro (robot description, xacro)
@@ -4,5 +4,32 @@
   <xacro:arg name="name" default="ur3e"/>
   <xacro:arg name="hande_name" default="robotiq_hande_gripper"/>
-   <!-- args for the hande -->
+  <!-- Extrusion -->
+  <!-- NOTE: this is for a right-mounted camera wrt robot base; maybe need to adjust rpy: 2.03 0.0 1.57 -->
+  <!-- Flip the sign for extrusion_x if your camera is mounted on the left; extrusion_z is the height of the camera optical axis from the table -->
+  <xacro:arg name="extrusion_x" default="0.566"/>
+  <xacro:arg name="extrusion_y" default="0.533"/>
+  <xacro:arg name="extrusion_z" default="0.467"/>
+  <xacro:arg name="extrusion_roll" default="0.0"/>
+  <xacro:arg name="extrusion_pitch" default="0.0"/>
+  <xacro:arg name="extrusion_yaw" default="0.0"/>
+  <xacro:arg name="cam_offset_x" default="0.02"/>
+  <xacro:arg name="cam_offset_y" default="0.0"/>
+  <xacro:arg name="cam_offset_z" default="0.01"/>
+  <xacro:arg name="cam_roll" default="0.0"/>
+  <xacro:arg name="cam_pitch" default="0.52"/>
+  <xacro:arg name="cam_yaw" default="-3.14"/>
+  <xacro:property name="cam_offset_x" value="$(arg cam_offset_x)"/>
+  <xacro:property name="cam_offset_y" value="$(arg cam_offset_y)"/>
+  <xacro:property name="cam_offset_z" value="$(arg cam_offset_z)"/>
+  <xacro:property name="cam_roll" value="$(arg cam_roll)"/>
+  <xacro:property name="cam_pitch" value="$(arg cam_pitch)"/>
+  <xacro:property name="cam_yaw" value="$(arg cam_yaw)"/>
+  <xacro:property name="extrusion_x" value="$(arg extrusion_x)"/>
+  <xacro:property name="extrusion_y" value="$(arg extrusion_y)"/>
+  <xacro:property name="extrusion_z" value="$(arg extrusion_z)"/>
+  <xacro:property name="extrusion_roll" value="$(arg extrusion_roll)"/>
+  <xacro:property name="extrusion_pitch" value="$(arg extrusion_pitch)"/>
+  <xacro:property name="extrusion_yaw" value="$(arg extrusion_yaw)"/>
+  <!-- args for the hande -->
   <xacro:arg name="parent" default="tool0"/>
   <xacro:arg name="grip_pos_min" default="0"/>
@@ -54,22 +81,8 @@
    <xacro:arg name="reverse_ip" default="0.0.0.0"/>
    <xacro:arg name="script_command_port" default="50004"/>
-   <!--   tool communication related parameters-->
-   <xacro:arg name="use_tool_communication" default="false" />
-   <xacro:arg name="tool_voltage" default="24" />
-   <xacro:arg name="tool_parity" default="N" />
-   <xacro:arg name="tool_baud_rate" default="115200" />
-   <xacro:arg name="tool_stop_bits" default="1" />
-   <xacro:arg name="tool_rx_idle_chars" default="1.5" />
-   <xacro:arg name="tool_tx_idle_chars" default="3.5" />
-   <xacro:arg name="tool_device_name" default="/tmp/ttyUR" />
-   <xacro:arg name="tool_tcp_port" default="54321" />
    <!--When using gazebo simulations absolute paths are necessary.-->
    <xacro:arg name="force_abs_paths" default="true" />
      <!-- Simulation parameters -->
-   <xacro:arg name="use_fake_hardware" default="true" />
-   <xacro:arg name="fake_sensor_commands" default="false" />
-   <xacro:arg name="sim_gazebo" default="false" />
-   <xacro:arg name="sim_ignition" default="false" />
-   <xacro:arg name="simulation_controllers" default="" />
+   <xacro:arg name="use_fake_hardware" default="false" />
    <!-- initial position for simulations (Fake Hardware, Gazebo, Ignition) -->
    <xacro:arg name="initial_positions_file" default="$(find ur_description)/config/initial_positions.yaml"/>
@@ -126,15 +139,4 @@
   <!-- Import table -->
   <xacro:include filename="$(find ur3e_hande_description)/urdf/table.urdf.xacro"/>
-  <!-- Import realsense -->
-  <xacro:if value="${is_import_ur3e and is_import_camera}">
-    <xacro:include filename="$(find realsense2_description)/urdf/_d435i.urdf.xacro"/>
-  </xacro:if>
-  <!-- Use the sensor_d435i macro; this is the camera on the right; add a unique namespace (e.g. camera2) if using both cameras-->
-  <xacro:if value="${is_import_ur3e and is_import_camera}">
-    <xacro:sensor_d435i parent="base_link">
-      <origin rpy="0 0.52 -3.14" xyz="0.546 0.533 0.467"/>   <!-- right camera -->
-      <!-- <origin rpy="0.0 0.698131 0" xyz="-0.522625 0.542925 0.3683"/>   --> <!-- left camera -->
-    </xacro:sensor_d435i>
-  </xacro:if>
   <!-- Joint between table and ur -->
   <xacro:if value="$(arg import_ur3e)">
@@ -145,11 +147,29 @@
     </joint>
   </xacro:if>
-  <!-- Joint between ur3e and hande -->
-<!-- <xacro:if value="${is_import_ur3e and is_import_hande}">
-  <joint name="ur3e_hande_joint" type="fixed">
-    <origin rpy="${pi/2} ${-pi/2} 0" xyz="0.00574 .03656 .01111"/>
-    <parent link="tool0"/>
-    <child link="robotiq_hande_coupler"/>
-  </joint>
-</xacro:if> -->
+  <!-- Include mount -->
+  <xacro:include filename="$(find ur3e_hande_description)/urdf/mounts/side_extrusion_mount.xacro"/>
+  <!-- Instantiate mount -->
+  <xacro:side_extrusion_20
+    parent="table"
+    x="$(arg extrusion_x)"
+    y="$(arg extrusion_y)"
+    z="$(arg extrusion_z)"
+    roll="$(arg extrusion_roll)"
+    pitch="$(arg extrusion_pitch)"
+    yaw="$(arg extrusion_yaw)"
+  />
+  <!-- Import realsense -->
+  <xacro:if value="${is_import_ur3e and is_import_camera}">
+    <xacro:include filename="$(find realsense2_description)/urdf/_d435i.urdf.xacro"/>
+  </xacro:if>
+  <!-- Use the sensor_d435i macro; this is the camera on the right -->
+  <!-- You must add a unique namespace (e.g. camera2) if using both multiple cameras -->
+  <xacro:if value="${is_import_ur3e and is_import_camera}">
+    <xacro:sensor_d435i parent="side_extrusion_20">
+      <origin
+      xyz="${cam_offset_x} ${cam_offset_y} ${cam_offset_z}"
+      rpy="${cam_roll} ${cam_pitch} ${cam_yaw}"
+      />
+    </xacro:sensor_d435i>
+  </xacro:if>
 </robot>
