Commit message: caps

File: src/hand_e/robotiq_hande_description/urdf_hw/robotiq_hande_gripper.urdf.xacro (robot description, xacro)
@@ -16,5 +16,5 @@
   <xacro:arg name="use_fake_hardware" default="true"/>
   <xacro:include filename="$(find robotiq_hande_description)/urdf_hw/robotiq_hande_gripper.xacro"/>
-  <!-- <link name="$(arg parent)"/> -->
+  <link name="$(arg parent)"/>
   <xacro:robotiq_hande_gripper
     name="robotiq_hande_gripper"

File: src/hand_e/robotiq_hande_description/urdf_hw/robotiq_hande_gripper.xacro (robot description, xacro)
@@ -22,5 +22,5 @@
             frequency_hz:=10
             create_socat_tty:=false
-            socat_ip_address:=192.168.100.10
+            socat_ip_address:=192.168.77.22
             socat_port:=54321
             coupler_mass:=0.119

File: src/ur3e_hande/ur3e_hande_description/urdf/ur3e.urdf.xacro (robot description, xacro)
@@ -1,9 +1,9 @@
 <?xml version="1.0"?>
-<robot xmlns:xacro="http://wiki.ros.org/xacro" name="ur">
+<robot xmlns:xacro="http://wiki.ros.org/xacro" name="$(arg name)">
    <!-- robot name parameter -->
    <xacro:arg name="name" default="ur"/>
    <!-- import main macro -->
    <xacro:include filename="$(find ur_description)/urdf/ur_macro.xacro"/>
-   <!-- possible 'ur_type' values: ur3, ur3e, ur5, ur5e, ur7e, ur10, ur10e, ur12e, ur16e, ur15, ur20, ur30 -->
+   <!-- possible 'ur_type' values: ur3, ur5, ur10, ur3e, ur5e, ur7e, ur10e, ur12e, ur16e, ur8long, ur15, ur18, ur20, ur30 -->
    <!-- the default value should raise an error in case this was called without defining the type -->
    <xacro:arg name="ur_type" default="ur3e"/>
@@ -11,5 +11,5 @@
    <xacro:arg name="tf_prefix" default="" />
    <xacro:arg name="joint_limit_params" default="$(find ur_description)/config/$(arg ur_type)/joint_limits.yaml"/>
-   <xacro:arg name="kinematics_params" default="$(find ur_description)/config/$(arg ur_type)/default_kinematics.yaml"/>
+   <xacro:arg name="kinematics_params" default="/home/robot/kinematic_config/ur3e_mrc.yaml"/>
    <xacro:arg name="physical_params" default="$(find ur_description)/config/$(arg ur_type)/physical_parameters.yaml"/>
    <xacro:arg name="visual_params" default="$(find ur_description)/config/$(arg ur_type)/visual_parameters.yaml"/>
@@ -19,5 +19,5 @@
    <xacro:arg name="safety_k_position" default="20"/>
    <!--When using gazebo simulations absolute paths are necessary.-->
-   <xacro:arg name="force_abs_paths" default="true" />
+   <xacro:arg name="force_abs_paths" default="false" />
    <!-- create link fixed to the "world" -->
    <link name="world" />

File: src/ur3e_hande/ur3e_hande_description/urdf/ur3e_hande_hw.urdf.xacro (robot description, xacro)
@@ -31,4 +31,5 @@
   <xacro:if value="$(arg import_ur3e)">
     <xacro:include filename="$(find ur_description)/urdf/ur_macro.xacro"/>
+    <xacro:include filename="$(find ur_description)/urdf/ros2_control_mock_hardware.xacro" />
   </xacro:if>
    <!-- possible 'ur_type' values: ur3, ur3e, ur5, ur5e, ur10, ur10e, ur16e -->
@@ -44,4 +45,5 @@
    <xacro:arg name="safety_pos_margin" default="0.15"/>
    <xacro:arg name="safety_k_position" default="20"/>
+   <xacro:arg name="mock_sensor_commands" default="false" />
    <!-- ros2_control related parameters -->
    <xacro:arg name="headless_mode" default="false" />
@@ -65,5 +67,5 @@
    <xacro:arg name="force_abs_paths" default="true" />
      <!-- Simulation parameters -->
-   <xacro:arg name="use_fake_hardware" default="false" />
+   <xacro:arg name="use_fake_hardware" default="true" />
    <xacro:arg name="fake_sensor_commands" default="false" />
    <xacro:arg name="sim_gazebo" default="false" />
@@ -94,4 +96,12 @@
    </xacro:ur_robot>
    </xacro:if>
+    <!-- ros2 control instance -->
+    <xacro:ur_ros2_control
+      name="$(arg name)"
+      tf_prefix="$(arg tf_prefix)"
+      mock_sensor_commands="$(arg mock_sensor_commands)"
+      initial_positions="${xacro.load_yaml(initial_positions_file)}"
+    />
+    <!-- Add tjhe hande -->
     <xacro:if value="$(arg import_hande)">
       <xacro:robotiq_hande_gripper
@@ -122,6 +132,6 @@
   <!-- Use the sensor_d435i macro; this is the camera on the right; add a unique namespace (e.g. camera2) if using both cameras-->
   <xacro:if value="${is_import_ur3e and is_import_camera}">
-    <xacro:sensor_d435i parent="world">
-      <origin rpy="0 0.52 0" xyz="-0.546 0.533 0.467"/>   <!-- right camera -->
+    <xacro:sensor_d435i parent="base_link">
+      <origin rpy="0 0.52 -3.14" xyz="0.546 0.533 0.467"/>   <!-- right camera -->
       <!-- <origin rpy="0.0 0.698131 0" xyz="-0.522625 0.542925 0.3683"/>   --> <!-- left camera -->
     </xacro:sensor_d435i>
