Commit message: pnp-v0

File: src/ur3e/ur3e_description/urdf/ur3e.urdf.xacro (robot description, xacro)
@@ -8,4 +8,31 @@
    <!-- the default value should raise an error in case this was called without defining the type -->
    <xacro:arg name="ur_type" default="ur3e"/>
+   <!-- Extrusion -->
+  <!-- NOTE: this is for a right-mounted camera wrt robot base; maybe need to adjust rpy: 2.03 0.0 1.57 -->
+  <!-- Flip the sign for extrusion_x if your camera is mounted on the left; extrusion_z is the height of the camera optical axis from the table -->
+  <xacro:arg name="extrusion_x" default="0.58"/>
+  <xacro:arg name="extrusion_y" default="0.533"/>
+  <xacro:arg name="extrusion_z" default="0.467"/>
+  <xacro:arg name="extrusion_roll" default="0.0"/>
+  <xacro:arg name="extrusion_pitch" default="0.0"/>
+  <xacro:arg name="extrusion_yaw" default="0.0"/>
+  <xacro:arg name="cam_offset_x" default="-0.005"/>
+  <xacro:arg name="cam_offset_y" default="0.0"/>
+  <xacro:arg name="cam_offset_z" default="0.0105"/>
+  <xacro:arg name="cam_roll" default="0.0"/>
+  <xacro:arg name="cam_pitch" default="0.32"/>
+  <xacro:arg name="cam_yaw" default="-3.14"/>
+  <xacro:property name="cam_offset_x" value="$(arg cam_offset_x)"/>
+  <xacro:property name="cam_offset_y" value="$(arg cam_offset_y)"/>
+  <xacro:property name="cam_offset_z" value="$(arg cam_offset_z)"/>
+  <xacro:property name="cam_roll" value="$(arg cam_roll)"/>
+  <xacro:property name="cam_pitch" value="$(arg cam_pitch)"/>
+  <xacro:property name="cam_yaw" value="$(arg cam_yaw)"/>
+  <xacro:property name="extrusion_x" value="$(arg extrusion_x)"/>
+  <xacro:property name="extrusion_y" value="$(arg extrusion_y)"/>
+  <xacro:property name="extrusion_z" value="$(arg extrusion_z)"/>
+  <xacro:property name="extrusion_roll" value="$(arg extrusion_roll)"/>
+  <xacro:property name="extrusion_pitch" value="$(arg extrusion_pitch)"/>
+  <xacro:property name="extrusion_yaw" value="$(arg extrusion_yaw)"/>
    <!-- parameters -->
    <xacro:arg name="tf_prefix" default="" />
@@ -115,5 +142,5 @@
      trajectory_port="$(arg trajectory_port)"
      >
-     <origin xyz="0 0 0" rpy="0 0 0" />          <!-- position robot in the world -->
+     <origin xyz="0 0 0.85" rpy="0 0 0" />          <!-- position robot in the world -->
    </xacro:ur_robot>
    <xacro:if value="$(arg sim_gazebo)">
@@ -139,5 +166,23 @@
   </xacro:if>
   <!-- Import table -->
-  <xacro:include filename="$(find ur3e_description)/urdf/table.urdf"/>
+   <xacro:include filename="$(find ur3e_description)/urdf/table.urdf.xacro"/>
+  <!-- Joint between table and ur -->
+  <joint name="table_joint" type="fixed">
+        <origin rpy="0 0 0" xyz="0 0 0"/>
+        <parent link="base_link"/>
+        <child link="table"/>
+    </joint>
+    <!-- Include mount -->
+  <xacro:include filename="$(find ur3e_description)/urdf/side_extrusion_20.urdf.xacro"/>
+  <!-- Instantiate mount -->
+  <xacro:side_extrusion_20
+    parent="table"
+    x="$(arg extrusion_x)"
+    y="$(arg extrusion_y)"
+    z="$(arg extrusion_z)"
+    roll="$(arg extrusion_roll)"
+    pitch="$(arg extrusion_pitch)"
+    yaw="$(arg extrusion_yaw)"
+  />
   <!-- Import realsense -->
   <xacro:include filename="$(find realsense2_description)/urdf/_d435i.urdf.xacro"/>
@@ -147,12 +192,9 @@
   </xacro:sensor_d435i> -->
   <!-- Use the sensor_d435i macro; this is the camera on the right; add a unique namespace (e.g. camera2) if using both cameras-->
-  <xacro:sensor_d435i parent="world">
-      <origin rpy="0.0 0.4712 0" xyz="-0.5762625 0.542925 0.40005"/>
+ <xacro:sensor_d435i parent="side_extrusion_20">
+      <origin
+      xyz="${cam_offset_x} ${cam_offset_y} ${cam_offset_z}"
+      rpy="${cam_roll} ${cam_pitch} ${cam_yaw}"
+      />
   </xacro:sensor_d435i>
-  <!-- Joint between table and ur -->
-  <joint name="table_joint" type="fixed">
-      <origin rpy="0 0 0" xyz="0 0 0"/>
-      <parent link="base_link"/>
-      <child link="table"/>
-  </joint>
 </robot>

File: src/ur3e_hande/ur3e_hande_description/urdf/ur3e_hande.urdf.xacro (robot description, xacro)
@@ -1,10 +1,11 @@
 <?xml version="1.0"?>
 <robot xmlns:xacro="http://www.ros.org/wiki/xacro" name="ur3e_hande">
-  <xacro:include filename="$(find robotiq_hande_description)/urdf/hande.urdf.xacro"/>
+  <!-- <xacro:include filename="$(find robotiq_hande_description)/urdf/hande.urdf.xacro"/> -->
+  <xacro:include filename="$(find robotiq_hande_description)/urdf/robotiq_hande_gripper.urdf.xacro"/>
   <xacro:include filename="$(find ur3e_description)/urdf/ur3e.urdf.xacro"/>
-  <joint name="ur3e_hande_joint" type="fixed">
+  <!-- <joint name="ur3e_hande_joint" type="fixed">
     <origin rpy="0 0 0" xyz="0 0 0"/>
     <parent link="tool0"/>
     <child link="robotiq_hande_coupler"/>
-  </joint>
+  </joint> -->
 </robot>

File: src/ur3e_hande/ur3e_hande_moveit_config/config/ur3e_hande.srdf.xacro (robot description, xacro)
@@ -49,7 +49,9 @@
   <group_state group="gripper" name="gripper_open">
     <joint name="robotiq_hande_left_finger_joint" value="0.025"/>
+    <joint name="robotiq_hande_right_finger_joint" value="0.025"/>
   </group_state>
   <group_state group="gripper" name="gripper_close">
     <joint name="robotiq_hande_left_finger_joint" value="0"/>
+    <joint name="robotiq_hande_right_finger_joint" value="0"/>
   </group_state>
   <!--END EFFECTOR: Purpose: Represent information about an end effector.-->
@@ -100,3 +102,28 @@
   <disable_collisions link1="wrist_1_link" link2="wrist_3_link" reason="Never"/>
   <disable_collisions link1="wrist_2_link" link2="wrist_3_link" reason="Adjacent"/>
+  <disable_collisions link1="base_link_inertia" link2="camera_link" reason="Never"/>
+    <disable_collisions link1="base_link_inertia" link2="shoulder_link" reason="Adjacent"/>
+    <disable_collisions link1="base_link_inertia" link2="side_extrusion_20" reason="Never"/>
+    <disable_collisions link1="base_link_inertia" link2="table" reason="Adjacent"/>
+    <disable_collisions link1="base_link_inertia" link2="upper_arm_link" reason="Never"/>
+    <disable_collisions link1="base_link_inertia" link2="wrist_1_link" reason="Never"/>
+    <disable_collisions link1="base_link_inertia" link2="wrist_2_link" reason="Never"/>
+    <disable_collisions link1="camera_link" link2="forearm_link" reason="Never"/>
+    <disable_collisions link1="camera_link" link2="robotiq_hande_coupler" reason="Never"/>
+    <disable_collisions link1="camera_link" link2="robotiq_hande_link" reason="Never"/>
+    <disable_collisions link1="camera_link" link2="shoulder_link" reason="Never"/>
+    <disable_collisions link1="camera_link" link2="side_extrusion_20" reason="Adjacent"/>
+    <disable_collisions link1="camera_link" link2="table" reason="Never"/>
+    <disable_collisions link1="camera_link" link2="upper_arm_link" reason="Never"/>
+    <disable_collisions link1="camera_link" link2="wrist_1_link" reason="Never"/>
+    <disable_collisions link1="camera_link" link2="wrist_2_link" reason="Never"/>
+    <disable_collisions link1="camera_link" link2="wrist_3_link" reason="Never"/>
+    <disable_collisions link1="forearm_link" link2="side_extrusion_20" reason="Never"/>
+    <disable_collisions link1="forearm_link" link2="upper_arm_link" reason="Adjacent"/>
+    <disable_collisions link1="forearm_link" link2="wrist_1_link" reason="Adjacent"/>
+    <disable_collisions link1="side_extrusion_20" link2="table" reason="Adjacent"/>
+    <disable_collisions link1="side_extrusion_20" link2="upper_arm_link" reason="Never"/>
+    <disable_collisions link1="side_extrusion_20" link2="wrist_1_link" reason="Never"/>
+    <disable_collisions link1="side_extrusion_20" link2="wrist_2_link" reason="Never"/>
+    <disable_collisions link1="side_extrusion_20" link2="wrist_3_link" reason="Never"/>
 </robot>

File: src/ur3e_hande/ur3e_hande_moveit_config/config/ur3e_hande.urdf.xacro (robot description, xacro)
@@ -2,8 +2,40 @@
 <robot xmlns:xacro="http://www.ros.org/wiki/xacro" name="name">
     <xacro:arg name="initial_positions_file" default="initial_positions.yaml" />
+    <xacro:arg name="parent" default="tool0"/>
+    <xacro:arg name="grip_pos_min" default="0"/>
+    <xacro:arg name="grip_pos_max" default="0.025"/>
+    <xacro:arg name="tty_port" default="/tmp/ttyUR"/>
+    <xacro:arg name="baudrate" default="115200"/>
+    <xacro:arg name="parity" default="N"/>
+    <xacro:arg name="data_bits" default="8"/>
+    <xacro:arg name="stop_bit" default="1"/>
+    <xacro:arg name="slave_id" default="9"/>
+    <xacro:arg name="frequency_hz" default="10"/>
+    <xacro:arg name="create_socat_tty" default="false"/>
+    <xacro:arg name="socat_ip_address" default="192.168.77.22"/>
+    <xacro:arg name="socat_port" default="54321"/>
+    <xacro:arg name="use_fake_hardware" default="true"/>
     <!-- Import name urdf file -->
     <xacro:include filename="$(find ur3e_hande_description)/urdf/ur3e_hande.urdf.xacro" />
+    <xacro:include filename="$(find robotiq_hande_description)/urdf/robotiq_hande_gripper.ros2_control.xacro"/>
     <!-- Import control_xacro -->
     <xacro:include filename="ur3e_hande.ros2_control.xacro" />
+    <xacro:robotiq_hande_ros2_control
+      name="${name}"
+      prefix="${prefix}"
+      grip_pos_min="${grip_pos_min}"
+      grip_pos_max="${grip_pos_max}"
+      tty_port="${tty_port}"
+      baudrate="${baudrate}"
+      parity="${parity}"
+      data_bits="${data_bits}"
+      stop_bit="${stop_bit}"
+      slave_id="${slave_id}"
+      frequency_hz="${frequency_hz}"
+      create_socat_tty="${create_socat_tty}"
+      socat_ip_address="${socat_ip_address}"
+      socat_port="${socat_port}"
+      use_fake_hardware="${use_fake_hardware}"
+    />
     <!-- HW interface in the works; NA for now -->
     <!-- <xacro:ur3e_hande_ros2_control name="robotiq_hande_controllers/RobotiqHandeHardwareInterface" initial_positions_file="$(arg initial_positions_file)"/> -->

Commit message: pnp-v0

File: src/ur3e/ur3e_description/urdf/ur3e.urdf.xacro (robot description, xacro)
@@ -13,9 +13,9 @@
   <xacro:arg name="extrusion_x" default="0.58"/>
   <xacro:arg name="extrusion_y" default="0.533"/>
-  <xacro:arg name="extrusion_z" default="0.467"/>
+  <xacro:arg name="extrusion_z" default="0.50"/>
   <xacro:arg name="extrusion_roll" default="0.0"/>
   <xacro:arg name="extrusion_pitch" default="0.0"/>
   <xacro:arg name="extrusion_yaw" default="0.0"/>
-  <xacro:arg name="cam_offset_x" default="-0.005"/>
+  <xacro:arg name="cam_offset_x" default="0.002"/>
   <xacro:arg name="cam_offset_y" default="0.0"/>
   <xacro:arg name="cam_offset_z" default="0.0105"/>
@@ -142,5 +142,5 @@
      trajectory_port="$(arg trajectory_port)"
      >
-     <origin xyz="0 0 0.85" rpy="0 0 0" />          <!-- position robot in the world -->
+     <origin xyz="0 0 0.7" rpy="0 0 0" />          <!-- position robot in the world -->
    </xacro:ur_robot>
    <xacro:if value="$(arg sim_gazebo)">
@@ -166,5 +166,5 @@
   </xacro:if>
   <!-- Import table -->
-   <xacro:include filename="$(find ur3e_description)/urdf/table.urdf.xacro"/>
+   <xacro:include filename="$(find ur3e_description)/urdf/table.urdf"/>
   <!-- Joint between table and ur -->
   <joint name="table_joint" type="fixed">
@@ -192,9 +192,18 @@
   </xacro:sensor_d435i> -->
   <!-- Use the sensor_d435i macro; this is the camera on the right; add a unique namespace (e.g. camera2) if using both cameras-->
- <xacro:sensor_d435i parent="side_extrusion_20">
+ <!-- <xacro:sensor_d435i parent="side_extrusion_20">
       <origin
       xyz="${cam_offset_x} ${cam_offset_y} ${cam_offset_z}"
       rpy="${cam_roll} ${cam_pitch} ${cam_yaw}"
       />
-  </xacro:sensor_d435i>
+  </xacro:sensor_d435i> -->
+  <xacro:sensor_d435i parent="base_link">
+        <origin rpy="0.0 0.5 -3.14" xyz="0.555 0.5333 0.467"/>
+    </xacro:sensor_d435i>
+  <link name="camera_optical_link"/>
+  <joint name="align_camera_joint" type="fixed">
+    <parent link="camera_link"/>
+    <child link="camera_optical_link"/>
+    <origin xyz="0 0 0" rpy="${-pi/2} 0 ${pi}"/> <!-- sim: -3.14 -1.57 1.57; recc: ${-pi/2} 0 ${-pi/2}-->
+  </joint>
 </robot>
